Commit message: chapter 14 code

File: ch10/nav2_mobile_robot/urdf/nav2_mobile_robot.xacro (robot description, xacro)
@@ -77,4 +77,31 @@
       <child link="lidar_link"/>
     </joint>
+  <link name="depth_link">
+    <visual>
+    <origin xyz="0 0 0.0" rpy="0 0 0"/>
+      <geometry>
+        <box size="0.05 0.05 0.05" />
+      </geometry>
+    </visual>
+    <collision>
+      <origin xyz="0 0 0.0" rpy="0 0 0"/>
+      <geometry>
+        <box size="0.05 0.05 0.05" />
+      </geometry>
+    </collision>
+    <inertial>
+      <origin xyz="0 0 0.0" rpy="0 0 0"/>
+      <mass value="1"/>
+      <inertia
+        ixx="1.0" ixy="0.0" ixz="0.0"
+        iyy="1.0" iyz="0.0"
+        izz="1.0"/>
+    </inertial>
+  </link>
+  <joint name='depth_link_joint' type='fixed'>
+    <origin xyz="0 0 0.1" rpy="0 0 0"/>
+    <parent link="base_link"/>
+    <child link="depth_link"/>
+  </joint>
 	  <gazebo reference="lidar_link">
         <sensor name="lidar" type='gpu_lidar'>
@@ -112,4 +139,59 @@
         </sensor>
     </gazebo>
+	  <gazebo reference="depth_link">
+        <xacro:include filename="$(find realsense2_description)/urdf/_d435.urdf.xacro"/>
+        <xacro:sensor_d435 parent="base_link" use_nominal_extrinsics="true" add_plug="false" use_mesh="true">
+            <origin xyz="0 0 0.5" rpy="0 0 0"/>
+        </xacro:sensor_d435>
+        <sensor name="cube_camera" type="camera">
+            <always_on>1</always_on>
+            <update_rate>30</update_rate>
+            <visualize>1</visualize>
+            <pose>0 0.0175 0.5125 0 -0 0</pose>
+            <topic>/camera/image_raw</topic>
+            <camera name="camera">
+                <horizontal_fov>1.48702</horizontal_fov>
+                <image>
+                    <width>1280</width>
+                    <height>720</height>
+                    <format>RGB_INT8</format>
+                </image>
+                <clip>
+                    <near>0.2</near>
+                    <far>10</far>
+                </clip>
+                <noise>
+                    <type>gaussian</type>
+                    <mean>0</mean>
+                    <stddev>0.007</stddev>
+                </noise>
+            </camera>
+        </sensor>
+        <sensor name='d435_depth' type='depth_camera'>
+            <ignition_frame_id>camera_link</ignition_frame_id>
+            <always_on>1</always_on>
+            <update_rate>30</update_rate>
+            <visualize>1</visualize>
+            <topic>/depth/image_raw</topic>
+            <pose>0 0.0175 0.5125 0 -0 0</pose>
+            <camera name='d435'>
+                <ignition_frame_id>camera_link</ignition_frame_id>
+                <horizontal_fov>1.48702</horizontal_fov>
+                <image>
+                    <width>1280</width>
+                    <height>720</height>
+                </image>
+                <clip>
+                    <near>0.2</near>
+                    <far>10</far>
+                </clip>
+                <noise>
+                    <type>gaussian</type>
+                    <mean>0</mean>
+                    <stddev>0.1</stddev>
+                </noise>
+            </camera>
+        </sensor>
+    </gazebo>
   <gazebo>
     <plugin filename="libignition-gazebo-odometry-publisher-system" name="ignition::gazebo::systems::OdometryPublisher">
